Commit message: ADD: mecanum gazebo velodyne simulation

File: src/mecanum_robot_description/urdf/mecanum_robot/mecanum.gazebo.xacro (robot description, xacro)
@@ -44,5 +44,5 @@
       <material>Gazebo/Grey</material>
     </gazebo>
-    <gazebo>
+    <!-- <gazebo>
       <plugin name="imu_plugin" filename="libgazebo_ros_imu.so">
         <alwaysOn>true</alwaysOn>
@@ -71,5 +71,5 @@
         </imu>
       </plugin>
-    </gazebo>
+    </gazebo> -->
     <!-- <gazebo reference="front_R_wheel">
       <mu1>1.0</mu1>
@@ -83,5 +83,5 @@
       <material>Gazebo/DarkGrey</material>
   </gazebo> -->
-    <gazebo reference="base_scan">
+    <!-- <gazebo reference="base_scan">
       <material>Gazebo/FlatBlack</material>
       <sensor type="ray" name="lds_lfcd_sensor">
@@ -114,6 +114,6 @@
         </plugin>
       </sensor>
-    </gazebo>
-    <gazebo reference="camera_link">
+    </gazebo> -->
+    <!-- <gazebo reference="camera_link">
       <sensor name="mecanum_camera_ir" type="depth">
         <update_rate>0</update_rate>
@@ -148,13 +148,13 @@
           <distortionT1>0.00000001</distortionT1>
           <distortionT2>0.00000001</distortionT2>
-          <!-- <CxPrime>0</CxPrime>
+          <CxPrime>0</CxPrime>
           <Cx>640</Cx>
           <Cy>360</Cy>
-          <focalLength>639.9976491530514</focalLength> -->
+          <focalLength>639.9976491530514</focalLength>
           <hackBaseline>0</hackBaseline>
         </plugin>
       </sensor>
     </gazebo>
-  </xacro:macro>
+  </xacro:macro> -->
   <!--gazebo>
    <plugin name="gazebo_grasp_fix" filename="libgazebo_grasp_fix.so">
@@ -175,3 +175,4 @@
     </plugin>
 </gazebo!-->
+  </xacro:macro>
 </robot>
