Commit message: EDIT: edit velodyne parameter

File: src/mecanum_robot_description/urdf/mecanum_robot_velodyne/mecanum.gazebo.xacro (robot description, xacro)
@@ -61,5 +61,5 @@
     </gazebo>
     <gazebo reference="velodyne">
-      <sensor type="ray" name="velodyne-VLP16">      <!-- ray   -->   <!-- gpu_ray -->
+      <sensor type="gpu_ray" name="velodyne-VLP16">      <!-- ray   -->   <!-- gpu_ray -->
         <pose>0 0 0 0 0 0</pose>
         <visualize>false</visualize>
@@ -68,8 +68,8 @@
           <scan>
             <horizontal>
-              <samples>1875</samples>
+              <samples>440</samples>
               <resolution>1</resolution>
-              <min_angle>0.9</min_angle>
-              <max_angle>130</max_angle>
+              <min_angle>-3.14</min_angle>
+              <max_angle>3.14</max_angle>
             </horizontal>
             <vertical>
@@ -81,5 +81,5 @@
           </scan>
           <range>
-            <min>0.9</min>
+            <min>0.3</min>
             <max>131</max>
             <resolution>0.001</resolution>
@@ -91,10 +91,10 @@
           </noise>
         </ray>
-        <plugin name="gazebo_ros_laser_controller" filename="libgazebo_ros_velodyne_laser.so">     <!-- libgazebo_ros_velodyne_gpu_laser  --> <!-- libgazebo_ros_velodyne_laser  -->
+        <plugin name="gazebo_ros_laser_controller" filename="libgazebo_ros_velodyne_gpu_laser.so">     <!-- libgazebo_ros_velodyne_gpu_laser  --> <!-- libgazebo_ros_velodyne_laser  -->
           <topicName>/velodyne_points</topicName>
           <frameName>velodyne</frameName>
           <organize_cloud>false</organize_cloud>
           <min_range>0.9</min_range>
-          <max_range>130</max_range>
+          <max_range>130.0</max_range>
           <gaussianNoise>0.008</gaussianNoise>
         </plugin>
@@ -102,14 +102,3 @@
     </gazebo>
   </xacro:macro>
-    <!-- <gazebo reference="front_R_wheel">
-      <mu1>1.0</mu1>
-      <mu2>1.0</mu2>
-      <kp>1e+13</kp>
-      <kd>1.0</kd>
-      <maxVel>0.001</maxVel>
-      <minDepth>0.00000000001</minDepth>
-      <turnGravityOff>false</turnGravityOff>
-      <gravity>1</gravity>
-      <material>Gazebo/DarkGrey</material>
-  </gazebo> -->
 </robot>

File: src/mecanum_robot_description/urdf/mecanum_robot_velodyne/mecanum_frame.urdf.xacro (robot description, xacro)
@@ -63,4 +63,11 @@
     </joint>
     <link name="VLP16_base_link">
+      <inertial>
+        <mass value="0.83"/>
+        <origin xyz="0 0 0.03585"/>
+        <inertia ixx="${(0.83 * (3.0*0.0516*0.0516 + 0.0717*0.0717)) / 12.0}" ixy="0" ixz="0"
+          iyy="${(0.83 * (3.0*0.0516*0.0516 + 0.0717*0.0717)) / 12.0}" iyz="0"
+          izz="${0.5 * 0.83 * (0.0516*0.0516)}"/>
+      </inertial>
       <visual>
         <geometry>
