Commit message: FIX: fix mecanum imu plugin

File: src/mecanum_robot_description/urdf/mecanum_robot_velodyne/cycloid_gear_mecanum_wheel.urdf.xacro (robot description, xacro)
@@ -71,6 +71,6 @@
         </transmission>
         <gazebo reference="${prefix}_wheel">
-            <mu1>1.0</mu1>
-            <mu2>1.0</mu2>
+            <mu1>0.0</mu1>
+            <mu2>0.0</mu2>
             <kp>1e+13</kp>
             <kd>1.0</kd>

File: src/mecanum_robot_description/urdf/mecanum_robot_velodyne/mecanum.gazebo.xacro (robot description, xacro)
@@ -13,5 +13,5 @@
   </gazebo>
   <gazebo>
-    <plugin name="$custom_controller" filename="libcustom_control_plugin.so">
+    <plugin name="custom_controller" filename="libcustom_control_plugin.so">
         <commandTopic>/mecanum_vel</commandTopic>
         <odometryTopic>/odom</odometryTopic>
@@ -23,10 +23,10 @@
   </xacro:macro>
   <xacro:macro name="sensor_gazebo" params="">
-    <gazebo reference="imu_link">
+    <!-- <gazebo reference="imu_link">
+      <gravity>true</gravity>
       <sensor type="imu" name="imu">
         <always_on>true</always_on>
         <visualize>false</visualize>
       </sensor>
-      <material>Gazebo/Grey</material>
     </gazebo>
     <gazebo>
@@ -57,4 +57,23 @@
         </imu>
       </plugin>
+    </gazebo> -->
+    <gazebo reference="imu_link">
+      <gravity>true</gravity>
+      <sensor name="imu_sensor" type="imu">
+        <always_on>true</always_on>
+        <update_rate>100</update_rate>
+        <visualize>true</visualize>
+        <topic>__default_topic__</topic>
+        <plugin filename="libgazebo_ros_imu_sensor.so" name="imu_plugin">
+          <topicName>imu</topicName>
+          <bodyName>imu_link</bodyName>
+          <updateRateHZ>200.0</updateRateHZ>
+          <gaussianNoise>0.0</gaussianNoise>
+          <xyzOffset>0 0 0</xyzOffset>
+          <rpyOffset>0 0 0</rpyOffset>
+          <frameName>imu_link</frameName>
+        </plugin>
+        <pose>0 0 0 0 0 0</pose>
+      </sensor>
     </gazebo>
     <gazebo reference="velodyne">
